File: pcb-esp32-tmc2209.kicad_sch (KiCad schematic)
At the start: 16 parts, among them J1 Conn_01x04_Pin, J2 12V Terminal, J3 5V Terminal, J4 Extra Pins, J5 Button 1, J6 Button 2, J7 PINHD_1x12_Male, J8 12V Output, U1 nanoESP32-C6

Commit message: initial commit of version 2
Parts:
- removed H4: MountingHole_M3, PCM_SL_Mechanical:MountingHole_3.2mm_Pad, symbol PCM_SL_Mechanical:MountingHole_M3_3.2mm_Pad
- removed J2: 12V Terminal, TerminalBlock_RND:TerminalBlock_RND_205-00276_1x02_P5.00mm_Vertical, symbol Connector:Screw_Terminal_01x02
- removed J3: 5V Terminal, TerminalBlock_RND:TerminalBlock_RND_205-00276_1x02_P5.00mm_Vertical, symbol Connector:Screw_Terminal_01x02
- removed J4: Extra Pins, Connector_PinHeader_2.54mm:PinHeader_1x02_P2.54mm_Vertical, symbol PCM_SL_Pin_Headers:PINHD_1x2_Male
- removed J5: Button 1, TerminalBlock_RND:TerminalBlock_RND_205-00276_1x02_P5.00mm_Vertical, symbol Connector:Screw_Terminal_01x02
- removed J6: Button 2, TerminalBlock_RND:TerminalBlock_RND_205-00276_1x02_P5.00mm_Vertical, symbol Connector:Screw_Terminal_01x02
- removed J7: PINHD_1x12_Male, Connector_PinHeader_2.54mm:PinHeader_1x12_P2.54mm_Vertical, symbol PCM_SL_Pin_Headers:PINHD_1x12_Male
- removed J8: 12V Output, Connector_PinHeader_2.54mm:PinHeader_1x02_P2.54mm_Vertical, symbol PCM_SL_Pin_Headers:PINHD_1x2_Male
- removed U2: ~, CustomComponents:BuckConverter, symbol CustomComponents:BuckConverter
- added J2: Screw_Terminal_8_P5.00mm, TerminalBlock:TerminalBlock_bornier-8_P5.08mm, symbol PCM_SL_Screw_Terminal:Screw_Terminal_8_P5.00mm
- added J3: PINHD_1x12_Female, Connector_PinSocket_2.54mm:PinSocket_1x12_P2.54mm_Vertical, symbol PCM_SL_Pin_Headers:PINHD_1x12_Female
- added J5: Microstep Selector, Connector_PinHeader_2.54mm:PinHeader_2x03_P2.54mm_Vertical, symbol PCM_SL_Pin_Headers:PINHD_2x3_Male
- added J6: PINHD_1x4_Female, Connector_PinSocket_2.54mm:PinSocket_1x04_P2.54mm_Vertical, symbol PCM_SL_Pin_Headers:PINHD_1x4_Female
- added U2: ~, CustomComponents:V100-EY9 DC-DC Converter, symbol CustomComponents:V100-EY9_DC-DC_Converter
Connections:
- net +12V: now also J2.3, U2.4 (VIN+)
- net GND: now also TMC2209.1 (GND_5V), U1.1 (GND), U1.16 (GND), U1.29 (GND), J2.2, J2.4, J2.6, J2.8, J5.5, J5.6, U2.2 (VOUT-), U2.5 (VIN-)
- net at U1.12 (11): now also J6.4
- net +5V: now reaches TMC2209.2 (5V), U1.15 (5V)
- net +5V: now also U1.30 (5V), J2.1, J5.1, J5.2, U2.1 (VOUT+)
- net at U1.17 (2): now also J3.1
- net at U1.26 (19): now also J3.10
- net at U1.27 (18): now also J3.11
- net at U1.28 (9): now also J3.12
- net at U1.18 (3): now also J3.2
- net at U1.19 (TX): now also J3.3
- net at U1.20 (RX): now also J3.4
- net at U1.21 (15): now also J3.5
- net at U1.22 (23): now also J3.6
- net at U1.23 (22): now also J3.7
- net at U1.24 (21): now also J3.8
- net at U1.25 (20): now also J3.9
- net at U1.10 (8): now also J6.2; no longer TMC2209.16 (EN)
- net at U1.11 (10): now also J6.3
- net at U1.13 (12): now also J2.5
- net at U1.14 (13): now also J2.7
- net at U1.8 (0): now also TMC2209.16 (EN); no longer TMC2209.14 (MS2)
- net at U1.9 (1): now also J6.1; no longer TMC2209.15 (MS1)
- new net: J5.3, TMC2209.15 (MS1)
- new net: J5.4, TMC2209.14 (MS2)
- no-connect marks 9 -> 7
